Commit message: Make repeaters smaller.

File: catkin_ws/src/stage_simulation/urdf/repeater.urdf.xacro (robot description, xacro)
@@ -3,7 +3,7 @@
   <link name="robot_$(arg name)/base_link">
     <visual>
-      <origin xyz="0 0 0.25" rpy="0 0 0"/>
+      <origin xyz="0 0 0.2" rpy="0 0 0"/>
       <geometry>
-        <box size="0.5 0.5 0.5"/>
+        <box size="0.2 0.2 0.4"/>
       </geometry>
       <material name="green">
